File: kicad/GenericControlBoard/GenericControlBoard.kicad_pcb (KiCad board)
At the start: 2 copper layers, 67 x 107 mm, 86 parts, among them J1 Conn_02x03_Counter_Clockwise, J10 RMC, J11 RMC, J12 Conn_01x04, J13 Conn_01x04, J14 Conn_01x04, J15 Conn_01x04, J16 Conn_01x04, J17 Conn_01x04, J18 Conn_01x04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

Commit message: fixname
Other:
- board text added: "GN"
- board text added: "GenericControlBoard v1 5V ~1A / 3.3V ~1A 4‑CAN‑Motor / 8‑Flex‑IO CAN Daisy‑Chain / UART/I2C"
- board text removed: "CH"
- board text removed: "GenericControlBoard v2 5V ~1A / 3.3V ~1A 4‑CAN‑Motor / 8‑Flex‑IO CAN Daisy‑Chain / UART/I2C"
Changed lines of the file:
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@@
 		(layer "Edge.Cuts")
 	)
-	(gr_text "GenericControlBoard v2\n5V ~1A / 3.3V ~1A\n4‑CAN‑Motor / 8‑Flex‑IO\nCAN Daisy‑Chain / UART/I2C"
+	(gr_text "GenericControlBoard v1\n5V ~1A / 3.3V ~1A\n4‑CAN‑Motor / 8‑Flex‑IO\nCAN Daisy‑Chain / UART/I2C"
 		(at 145 142.3 0)
 		(layer "F.SilkS")
@@
 		)
 	)
-	(gr_text "GND"
-		(at 169.1 122 0)
+	(gr_text "GN"
+		(at 170.1 122 0)
 		(layer "F.SilkS" knockout)
 		(effects
@@
 		)
 	)
-	(gr_text "GND"
-		(at 126.7 57.8 0)
+	(gr_text "5V"
+		(at 127.7 57.8 0)
 		(layer "F.SilkS")
 		(effects
@@
 		)
 	)
-	(gr_text "+5V"
-		(at 168.9 129.4 0)
+	(gr_text "5V"
+		(at 170.138095 129.4 0)
 		(layer "F.SilkS" knockout)
 		(effects
@@
 		)
 	)
-	(gr_text "CH"
+	(gr_text "CL"
 		(at 170.138095 124.466667 0)
 		(layer "F.SilkS" knockout)
@@
 		)
 	)
-	(gr_text "5V"
-		(at 127.7 63 0)
-		(layer "F.SilkS")
-		(effects
+	(gr_text "GND"
+		(at 126.6 63 0)
+		(layer "F.SilkS")
+		(effects
